File: wled-pcb/wled-pcb.kicad_sch (KiCad schematic)
At the start: 28 parts, among them J2 Conn_02x03_Counter_Clockwise, J3 Screw_Terminal_01x03, J4 Screw_Terminal_01x03, J5 Screw_Terminal_01x03, J6 Screw_Terminal_01x02, J7 Screw_Terminal_01x03, K1 Relay_SPDT, Q1 BC337, U1 ESP32-DevKitC, U2 74125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

Commit message: add footprints
Parts:
- C1: footprint (none) -> Capacitor_THT:CP_Radial_D13.0mm_P5.00mm
- D2, D3, D4: footprint (none) -> LED_THT:LED_D5.0mm
- F1, F2, F3, F4: footprint (none) -> Fuse:Fuseholder_Blade_Mini_Keystone_3568
- J2: footprint (none) -> Package_DIP:DIP-6_W7.62mm_LongPads
- J3, J4, J5, J7: footprint (none) -> TerminalBlock:TerminalBlock_bornier-3_P5.08mm
- J6: footprint (none) -> TerminalBlock:TerminalBlock_bornier-2_P5.08mm
- R1, R2, R3, R4, R5, R6, R7, R8: footprint (none) -> Resistor_THT:R_Axial_DIN0207_L6.3mm_D2.5mm_P10.16mm_Horizontal
- U2: footprint (none) -> Package_DIP:DIP-14_W7.62mm_LongPads
Changed lines of the file:
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@@
       (effects (font (size 1.27 1.27)) (justify left))
     )
-    (property "Footprint" "" (at 187.96 55.88 0)
+    (property "Footprint" "TerminalBlock:TerminalBlock_bornier-3_P5.08mm" (at 187.96 55.88 0)
       (effects (font (size 1.27 1.27)) hide)
     )
@@
       (effects (font (size 1.27 1.27)))
     )
-    (property "Footprint" "" (at 175.26 55.118 90)
+    (property "Footprint" "Fuse:Fuseholder_Blade_Mini_Keystone_3568" (at 175.26 55.118 90)
       (effects (font (size 1.27 1.27)) hide)
     )
@@
       (effects (font (size 1.27 1.27)))
     )
-    (property "Footprint" "" (at 96.52 36.83 0)
+    (property "Footprint" "LED_THT:LED_D5.0mm" (at 96.52 36.83 0)
       (effects (font (size 1.27 1.27)) hide)
     )
@@
       (effects (font (size 1.27 1.27)))
     )
-    (property "Footprint" "" (at 246.38 82.042 90)
+    (property "Footprint" "Resistor_THT:R_Axial_DIN0207_L6.3mm_D2.5mm_P10.16mm_Horizontal" (at 246.38 82.042 90)
       (effects (font (size 1.27 1.27)) hide)
     )
@@
       (effects (font (size 1.27 1.27)))
     )
-    (property "Footprint" "" (at 175.26 94.488 90)
+    (property "Footprint" "Fuse:Fuseholder_Blade_Mini_Keystone_3568" (at 175.26 94.488 90)
       (effects (font (size 1.27 1.27)) hide)
     )
@@
       (effects (font (size 1.27 1.27)))
     )
-    (property "Footprint" "" (at 246.38 42.672 90)
+    (property "Footprint" "Resistor_THT:R_Axial_DIN0207_L6.3mm_D2.5mm_P10.16mm_Horizontal" (at 246.38 42.672 90)
       (effects (font (size 1.27 1.27)) hide)
     )
@@
       (effects (font (size 1.27 1.27)))
     )
-    (property "Footprint" "" (at 86.36 29.718 90)
+    (property "Footprint" "Resistor_THT:R_Axial_DIN0207_L6.3mm_D2.5mm_P10.16mm_Horizontal" (at 86.36 29.718 90)
       (effects (font (size 1.27 1.27)) hide)
     )
@@
       (effects (font (size 1.27 1.27)) (justify right))
     )
-    (property "Footprint" "" (at 98.298 165.1 90)
+    (property "Footprint" "Resistor_THT:R_Axial_DIN0207_L6.3mm_D2.5mm_P10.16mm_Horizontal" (at 98.298 165.1 90)
       (effects (font (size 1.27 1.27)) hide)
     )
@@
       (effects (font (size 1.27 1.27)) (justify left))
     )
-    (property "Footprint" "" (at 256.54 55.88 0)
+    (property "Footprint" "TerminalBlock:TerminalBlock_bornier-3_P5.08mm" (at 256.54 55.88 0)
       (effects (font (size 1.27 1.27)) hide)
     )
@@
       (effects (font (size 1.27 1.27)))
     )
-    (property "Footprint" "" (at 86.36 38.608 90)
+    (property "Footprint" "Resistor_THT:R_Axial_DIN0207_L6.3mm_D2.5mm_P10.16mm_Horizontal" (at 86.36 38.608 90)
       (effects (font (size 1.27 1.27)) hide)
     )
@@
       (effects (font (size 1.27 1.27)))
     )
-    (property "Footprint" "" (at 73.66 154.178 90)
+    (property "Footprint" "Resistor_THT:R_Axial_DIN0207_L6.3mm_D2.5mm_P10.16mm_Horizontal" (at 73.66 154.178 90)
       (effects (font (size 1.27 1.27)) hide)
     )
@@
       (effects (font (size 1.27 1.27)))
     )
-    (property "Footprint" "" (at 179.07 42.672 90)
+    (property "Footprint" "Resistor_THT:R_Axial_DIN0207_L6.3mm_D2.5mm_P10.16mm_Horizontal" (at 179.07 42.672 90)
       (effects (font (size 1.27 1.27)) hide)
     )
@@
       (effects (font (size 1.27 1.27)) (justify left))
     )
-    (property "Footprint" "" (at 256.54 95.25 0)
+    (property "Footprint" "TerminalBlock:TerminalBlock_bornier-3_P5.08mm" (at 256.54 95.25 0)
       (effects (font (size 1.27 1.27)) hide)
     )
@@
       (effects (font (size 1.27 1.27)))
     )
-    (property "Footprint" "" (at 227.33 44.45 0)
+    (property "Footprint" "Package_DIP:DIP-14_W7.62mm_LongPads" (at 227.33 44.45 0)
       (effects (font (size 1.27 1.27)) hide)
     )
@@
       (effects (font (size 1.27 1.27)))
     )
-    (property "Footprint" "" (at 227.33 83.82 0)
+    (property "Footprint" "Package_DIP:DIP-14_W7.62mm_LongPads" (at 227.33 83.82 0)
       (effects (font (size 1.27 1.27)) hide)
     )
@@
       (effects (font (size 1.27 1.27)))
     )
-    (property "Footprint" "" (at 96.52 27.94 0)
+    (property "Footprint" "LED_THT:LED_D5.0mm" (at 96.52 27.94 0)
       (effects (font (size 1.27 1.27)) hide)
     )
@@
       (effects (font (size 1.27 1.27)))
     )
-    (property "Footprint" "" (at 160.02 44.45 0)
+    (property "Footprint" "Package_DIP:DIP-14_W7.62mm_LongPads" (at 160.02 44.45 0)
       (effects (font (size 1.27 1.27)) hide)
     )
@@
       (effects (font (size 1.27 1.27)))
     )
-    (property "Footprint" "" (at 160.02 83.82 0)
+    (property "Footprint" "Package_DIP:DIP-14_W7.62mm_LongPads" (at 160.02 83.82 0)
       (effects (font (size 1.27 1.27)) hide)
     )
@@
       (effects (font (size 1.27 1.27)))
     )
-    (property "Footprint" "" (at 243.84 55.118 90)
+    (property "Footprint" "Fuse:Fuseholder_Blade_Mini_Keystone_3568" (at 243.84 55.118 90)
       (effects (font (size 1.27 1.27)) hide)
     )
@@
       (effects (font (size 1.27 1.27)))
     )
-    (property "Footprint" "" (at 179.07 82.042 90)
+    (property "Footprint" "Resistor_THT:R_Axial_DIN0207_L6.3mm_D2.5mm_P10.16mm_Horizontal" (at 179.07 82.042 90)
       (effects (font (size 1.27 1.27)) hide)
     )
@@
       (effects (font (size 1.27 1.27)))
     )
-    (property "Footprint" "" (at 243.84 94.488 90)
+    (property "Footprint" "Fuse:Fuseholder_Blade_Mini_Keystone_3568" (at 243.84 94.488 90)
       (effects (font (size 1.27 1.27)) hide)
     )
@@
       (effects (font (size 1.27 1.27)) (justify left))
     )
-    (property "Footprint" "" (at 51.7652 31.75 0)
+    (property "Footprint" "Capacitor_THT:CP_Radial_D13.0mm_P5.00mm" (at 51.7652 31.75 0)
       (effects (font (size 1.27 1.27)) hide)
     )
@@
       (effects (font (size 1.27 1.27)))
     )
-    (property "Footprint" "" (at 73.66 157.48 0)
+    (property "Footprint" "LED_THT:LED_D5.0mm" (at 73.66 157.48 0)
       (effects (font (size 1.27 1.27)) hide)
     )
@@
       (effects (font (size 1.27 1.27)))
     )
-    (property "Footprint" "" (at 224.79 143.51 0)
+    (property "Footprint" "Package_DIP:DIP-6_W7.62mm_LongPads" (at 224.79 143.51 0)
       (effects (font (size 1.27 1.27)) hide)
     )
@@
       (effects (font (size 1.27 1.27)) (justify left))
     )
-    (property "Footprint" "" (at 187.96 95.25 0)
+    (property "Footprint" "TerminalBlock:TerminalBlock_bornier-3_P5.08mm" (at 187.96 95.25 0)
       (effects (font (size 1.27 1.27)) hide)
     )
@@
       (effects (font (size 1.27 1.27)))
     )
-    (property "Footprint" "" (at 27.94 29.21 0)
-      (effects (font (size 1.27 1.27)) hide)
-    )
+    (property "Footprint" "TerminalBlock:TerminalBlock_bornier-2_P5.08mm" (at 27.94 29.21 0)
+      (effects (font (size 1.27 1.27)) hide)
+    )

Commit message: add footprints to pcb
Parts:
- K1: footprint (none) -> Relay_THT:Relay_SPDT_Omron_G2RL-1-E
Connections:
- net +3.3V: now also U3.1; no longer R6.1
- net +5V: now also J6.1 (Pin_1); no longer J6.2 (Pin_2)
- net GND: now also J6.2 (Pin_2); no longer J6.1 (Pin_1)
- net at R6.2: now also U3.2; no longer U3.1
- net at D3.2 (A): now also R6.1; no longer U3.2
Other:
- moved on the sheet: C1, D3, J6, R6

Commit message: fix some mistakes, route some traces
Connections:
- net led1 lo: now also U1.27 (GPIO16); no longer U1.20 (SD_CLK/GPIO6)
- net led2 lo: now also U1.28 (GPIO17); no longer U1.21 (SD_DATA0/GPIO7), U1.22 (SD_DATA1/GPIO8)
- net led3 lo: now also U1.30 (GPIO18)
- net led4 lo: now also U1.31 (GPIO19); no longer U1.16 (SD_DATA2/GPIO9)
- net at U3.2: now also R6.1; no longer R6.2
- net at D3.2 (A): now also R6.2; no longer R6.1
Other:
- moved on the sheet: R6
Changed lines of the file:
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@@
     (stroke (width 0) (type default))
   )
-  (wire (pts (xy 99.06 100.33) (xy 107.95 100.33))
-    (stroke (width 0) (type default))
-  )
-  (wire (pts (xy 99.06 102.87) (xy 107.95 102.87))
+  (wire (pts (xy 99.06 115.57) (xy 107.95 115.57))
+    (stroke (width 0) (type default))
+  )
+  (wire (pts (xy 99.06 118.11) (xy 107.95 118.11))
     (stroke (width 0) (type default))
   )
@@
     (stroke (width 0) (type default))
   )
-  (wire (pts (xy 99.06 105.41) (xy 107.95 105.41))
+  (wire (pts (xy 99.06 74.93) (xy 107.95 74.93))
     (stroke (width 0) (type default))
   )
@@
     (stroke (width 0) (type default))
   )
-  (wire (pts (xy 99.06 107.95) (xy 107.95 107.95))
+  (wire (pts (xy 99.06 77.47) (xy 107.95 77.47))
     (stroke (width 0) (type default))
   )
@@
     (effects (font (size 1.27 1.27)) (justify left bottom))
   )
-  (label "led4 lo" (at 107.95 107.95 0) (fields_autoplaced)
-    (effects (font (size 1.27 1.27)) (justify left bottom))
-  )
-  (label "led2 lo" (at 107.95 105.41 0) (fields_autoplaced)
+  (label "led4 lo" (at 107.95 77.47 0) (fields_autoplaced)
+    (effects (font (size 1.27 1.27)) (justify left bottom))
+  )
+  (label "led3 lo" (at 107.95 74.93 0) (fields_autoplaced)
     (effects (font (size 1.27 1.27)) (justify left bottom))
   )
@@
     (effects (font (size 1.27 1.27)) (justify right bottom))
   )
-  (label "led2 lo" (at 107.95 102.87 0) (fields_autoplaced)
+  (label "led2 lo" (at 107.95 118.11 0) (fields_autoplaced)
     (effects (font (size 1.27 1.27)) (justify left bottom))
   )
@@
     (effects (font (size 1.27 1.27)) (justify right bottom))
   )
-  (label "led1 lo" (at 107.95 100.33 0) (fields_autoplaced)
+  (label "led1 lo" (at 107.95 115.57 0) (fields_autoplaced)
     (effects (font (size 1.27 1.27)) (justify left bottom))
   )
@@
     )
   )
-  (symbol (lib_id "Device:R") (at 77.47 157.48 90) (unit 1)
+  (symbol (lib_id "Device:R") (at 77.47 157.48 270) (unit 1)
     (in_bom yes) (on_board yes) (dnp no) (fields_autoplaced)
     (property "Reference" "R6" (at 77.47 151.13 90)
@@
       (effects (font (size 1.27 1.27)))
     )
-    (property "Footprint" "Resistor_THT:R_Axial_DIN0207_L6.3mm_D2.5mm_P10.16mm_Horizontal" (at 77.47 159.258 90)
-      (effects (font (size 1.27 1.27)) hide)
-    )
+    (property "Footprint" "Resistor_THT:R_Axial_DIN0207_L6.3mm_D2.5mm_P10.16mm_Horizontal" (at 77.47 155.702 90)
+      (effects (font (size 1.27 1.27)) hide)
+    )

Commit message: Add buttons, route tracks
Parts:
- added H1, H2, H3, H4: MountingHole, MountingHole:MountingHole_3.2mm_M3_DIN965_Pad_TopBottom, symbol Mechanical:MountingHole
- added R10, R9: 10k, Resistor_THT:R_Axial_DIN0207_L6.3mm_D2.5mm_P10.16mm_Horizontal, symbol Device:R
- added SW1, SW2: SW_Push, Connector_PinHeader_2.54mm:PinHeader_1x02_P2.54mm_Vertical, symbol Switch:SW_Push
Connections:
- net +3.3V: now also R10.2, R9.2
- net GND: now also SW1.2, SW2.2
- net sw 1: now reaches U1.21 (SD_DATA0/GPIO7)
- net sw 1: now also R9.1, SW1.1
- net sw 2: now reaches U1.22 (SD_DATA1/GPIO8)
- net sw 2: now also R10.1, SW2.1

Commit message: layout board smaller than 100x100
Parts:
- SW1, SW2: footprint Connector_PinHeader_2.54mm:PinHeader_1x02_P2.54mm_Vertical -> Button_Switch_THT:SW_PUSH-12mm_Wuerth-430476085716
Changed lines of the file:
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@@
       (effects (font (size 1.27 1.27)))
     )
-    (property "Footprint" "Connector_PinHeader_2.54mm:PinHeader_1x02_P2.54mm_Vertical" (at 201.93 114.3 0)
+    (property "Footprint" "Button_Switch_THT:SW_PUSH-12mm_Wuerth-430476085716" (at 201.93 114.3 0)
       (effects (font (size 1.27 1.27)) hide)
     )
@@
       (effects (font (size 1.27 1.27)))
     )
-    (property "Footprint" "Connector_PinHeader_2.54mm:PinHeader_1x02_P2.54mm_Vertical" (at 153.67 114.3 0)
-      (effects (font (size 1.27 1.27)) hide)
-    )
+    (property "Footprint" "Button_Switch_THT:SW_PUSH-12mm_Wuerth-430476085716" (at 153.67 114.3 0)
+      (effects (font (size 1.27 1.27)) hide)
+    )

Commit message: use different pins for switches
Connections:
- net sw 1: now also U1.24 (ADC2_CH2/GPIO2); no longer U1.21 (SD_DATA0/GPIO7)
- net sw 2: now also U1.26 (ADC2_CH0/GPIO4); no longer U1.22 (SD_DATA1/GPIO8)
Changed lines of the file:
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@@
     (stroke (width 0) (type default))
   )
-  (wire (pts (xy 99.06 102.87) (xy 107.95 102.87))
+  (wire (pts (xy 99.06 67.31) (xy 107.95 67.31))
     (stroke (width 0) (type default))
   )
@@
     (stroke (width 0) (type default))
   )
-  (wire (pts (xy 99.06 105.41) (xy 107.95 105.41))
+  (wire (pts (xy 99.06 69.85) (xy 107.95 69.85))
     (stroke (width 0) (type default))
   )
@@
     (effects (font (size 1.27 1.27)) (justify right bottom))
   )
-  (label "sw 1" (at 107.95 102.87 0) (fields_autoplaced)
+  (label "sw 1" (at 107.95 67.31 0) (fields_autoplaced)
     (effects (font (size 1.27 1.27)) (justify left bottom))
   )
@@
     (effects (font (size 1.27 1.27)) (justify right bottom))
   )
-  (label "sw 2" (at 107.95 105.41 0) (fields_autoplaced)
-    (effects (font (size 1.27 1.27)) (justify left bottom))
-  )
+  (label "sw 2" (at 107.95 69.85 0) (fields_autoplaced)
+    (effects (font (size 1.27 1.27)) (justify left bottom))
+  )

Commit message: Add more info to silkscreen
Parts:
- R5, R8: value 150R -> 1K
- R6: value R -> 150R
- R7: value R -> 1K
Changed lines of the file:
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@@
       (effects (font (size 1.27 1.27)))
     )
-    (property "Value" "150R" (at 86.36 24.13 90)
+    (property "Value" "1K" (at 86.36 24.13 90)
       (effects (font (size 1.27 1.27)))
     )
@@
       (effects (font (size 1.27 1.27)) (justify right))
     )
-    (property "Value" "R" (at 99.06 166.37 0)
+    (property "Value" "1K" (at 99.06 166.37 0)
       (effects (font (size 1.27 1.27)) (justify right))
     )
@@
       (effects (font (size 1.27 1.27)))
     )
-    (property "Value" "150R" (at 86.36 33.02 90)
+    (property "Value" "1K" (at 86.36 33.02 90)
       (effects (font (size 1.27 1.27)))
     )
@@
       (effects (font (size 1.27 1.27)))
     )
-    (property "Value" "R" (at 77.47 153.67 90)
+    (property "Value" "150R" (at 77.47 153.67 90)
       (effects (font (size 1.27 1.27)))
     )
